Commit message: updated

File: description/robot.urdf.xacro (robot description, xacro)
@@ -2,3 +2,6 @@
 <robot xmlns:xacro="http://www.ros.org/wiki/xacro"  name="robot">
     <xacro:include filename="robot_core.xacro"/>
+    <xacro:include filename="gazebo_control.xacro"/>
+    <!--<xacro:include filename="camera.xacro"/>-->
+    <!--<xacro:include filename="depth_camera.xacro"/>-->
 </robot>

File: description/robot_core.xacro (robot description, xacro)
@@ -2,4 +2,5 @@
 <robot xmlns:xacro="http://www.ros.org/wiki/xacro">
     <xacro:include filename="inertial_macros.xacro"/>
+    <!-- [Keep all your material definitions - same as before] -->
     <material name="white">
         <color rgba="1 1 1 1" />
@@ -13,4 +14,28 @@
     <material name="black">
         <color rgba="0 0 0 1"/>
+    </material>
+    <material name="grey">
+        <color rgba="0.7 0.7 0.7 1"/>
+    </material>
+    <material name="peacock_blue">
+        <color rgba="0.0 0.4 0.6 1"/>
+    </material>
+    <material name="peacock_green">
+        <color rgba="0.0 0.5 0.4 1"/>
+    </material>
+    <material name="peacock_dark_blue">
+        <color rgba="0.0 0.2 0.4 1"/>
+    </material>
+    <material name="peacock_teal">
+        <color rgba="0.0 0.5 0.5 1"/>
+    </material>
+    <material name="peacock_gold">
+        <color rgba="0.85 0.65 0.13 1"/>
+    </material>
+    <material name="peacock_purple">
+        <color rgba="0.5 0.0 0.5 1"/>
+    </material>
+    <material name="peacock_turquoise">
+        <color rgba="0.25 0.88 0.82 1"/>
     </material>
     <!-- BASE LINK-->
@@ -21,29 +46,32 @@
         <parent link="base_link"/>
         <child link="chassis"/>
-        <origin xyz="-0.11 0 0.04"/>
+        <origin xyz="-0.125 0 0.015"/>
     </joint>
     <link name="chassis">
         <visual>
-            <origin xyz="0.11 0 0.075"/>
-            <geometry>
-                <cylinder radius="0.11" length="0.15"/>
-            </geometry>
-            <material name="orange"/>
-        </visual>
-        <collision>
-            <origin xyz="0.11 0 0.075"/>
-            <geometry>
-                <cylinder radius="0.11" length="0.15"/>
-            </geometry>
-        </collision>
-        <xacro:inertial_cylinder mass="0.5" radius="0.11" length="0.15">
-            <origin xyz="0.11 0 0.075" rpy="0 0 0"/>
-        </xacro:inertial_cylinder>
-    </link>
+            <origin xyz="0.125 0 0.0015"/>
+            <geometry>
+                <cylinder radius="0.125" length="0.003"/>
+            </geometry>
+            <material name="peacock_blue"/>
+        </visual>
+        <collision>
+            <origin xyz="0.125 0 0.0015"/>
+            <geometry>
+                <cylinder radius="0.125" length="0.003"/>
+            </geometry>
+        </collision>
+        <xacro:inertial_cylinder mass="1.5" radius="0.125" length="0.003">
+            <origin xyz="0.14 0 -0.01" rpy="0 0 0"/>
+        </xacro:inertial_cylinder>
+    </link>
+    <gazebo reference="chassis">
+        <material>Gazebo/Blue</material>
+    </gazebo>
     <!--LEFT WHEEL LINK-->
     <joint name="left_wheel_joint" type="continuous">
-        <parent link = "chassis"/>
-        <child link = "left_wheel"/>
-        <origin xyz="0.11 0.13 0" rpy="-1.5708 0 0"/>
+        <parent link="chassis"/>
+        <child link="left_wheel"/>
+        <origin xyz="0.125 0.13 0" rpy="-1.5708 0 0"/>
         <axis xyz="0 0 1"/>
     </joint>
@@ -51,22 +79,29 @@
         <visual>
             <geometry>
-                <cylinder radius="0.04" length="0.04"/>
-            </geometry>
-            <material name="black"/>
-        </visual>
-        <collision>
-            <geometry>
-                <cylinder radius="0.04" length="0.04"/>
-            </geometry>
-        </collision>
-        <xacro:inertial_cylinder mass="0.1" radius="0.04" length="0.04">
-            <origin xyz="0 0 0" rpy="0 0 0"/>
-        </xacro:inertial_cylinder>
-    </link>
+                <cylinder radius="0.035" length="0.04"/>
+            </geometry>
+            <material name="peacock_dark_blue"/>
+        </visual>
+        <collision>
+            <geometry>
+                <cylinder radius="0.035" length="0.04"/>
+            </geometry>
+        </collision>
+        <xacro:inertial_cylinder mass="0.15" radius="0.035" length="0.04">
+            <origin xyz="0 0 0" rpy="0 0 0"/>
+        </xacro:inertial_cylinder>
+    </link>
+    <gazebo reference="left_wheel">
+        <material>Gazebo/Purple</material>
+        <mu1>1.2</mu1>
+        <mu2>1.2</mu2>
+        <kp>1000000.0</kp>
+        <kd>100.0</kd>
+    </gazebo>
     <!--RIGHT WHEEL LINK-->
     <joint name="right_wheel_joint" type="continuous">
-        <parent link = "chassis"/>
-        <child link = "right_wheel"/>
-        <origin xyz="0.11 -0.13 0" rpy="1.5708 0 0"/>
+        <parent link="chassis"/>
+        <child link="right_wheel"/>
+        <origin xyz="0.125 -0.13 0" rpy="1.5708 0 0"/>
         <axis xyz="0 0 -1"/>
     </joint>
@@ -74,60 +109,274 @@
         <visual>
             <geometry>
-                <cylinder radius="0.04" length="0.04"/>
-            </geometry>
-            <material name="black"/>
-        </visual>
-        <collision>
-            <geometry>
-                <cylinder radius="0.04" length="0.04"/>
-            </geometry>
-        </collision>
-        <xacro:inertial_cylinder mass="0.1" radius="0.04" length="0.04">
-            <origin xyz="0 0 0" rpy="0 0 0"/>
-        </xacro:inertial_cylinder>
-    </link>
-    <!--CASTER WHEEL LINK1-->
+                <cylinder radius="0.035" length="0.04"/>
+            </geometry>
+            <material name="peacock_dark_blue"/>
+        </visual>
+        <collision>
+            <geometry>
+                <cylinder radius="0.035" length="0.04"/>
+            </geometry>
+        </collision>
+        <xacro:inertial_cylinder mass="0.15" radius="0.035" length="0.04">
+            <origin xyz="0 0 0" rpy="0 0 0"/>
+        </xacro:inertial_cylinder>
+    </link>
+    <gazebo reference="right_wheel">
+        <material>Gazebo/Purple</material>
+        <mu1>1.2</mu1>
+        <mu2>1.2</mu2>
+        <kp>1000000.0</kp>
+        <kd>100.0</kd>
+    </gazebo>
+    <!--CASTER SPACER 1 - Small cylinder to drop caster down-->
+    <joint name="caster_spacer_joint1" type="fixed">
+        <parent link="chassis"/>
+        <child link="caster_spacer1"/>
+        <origin xyz="0.025 0 -0.0075"/>
+    </joint>
+    <link name="caster_spacer1">
+        <visual>
+            <geometry>
+                <cylinder radius="0.003" length="0.02"/>  <!-- Small spacer: 3mm radius, 20mm length -->
+            </geometry>
+            <material name="grey"/>
+        </visual>
+        <collision>
+            <geometry>
+                <cylinder radius="0.003" length="0.02"/>
+            </geometry>
+        </collision>
+        <xacro:inertial_cylinder mass="0.01" radius="0.003" length="0.02">
+            <origin xyz="0 0 0" rpy="0 0 0"/>
+        </xacro:inertial_cylinder>
+    </link>
+    <gazebo reference="caster_spacer1">
+        <material>Gazebo/Grey</material>
+    </gazebo>
+    <!--CASTER WHEEL LINK1 - Attached to bottom of spacer-->
     <joint name="caster_wheel_joint1" type="fixed">
-        <parent link="chassis"/>
+        <parent link="caster_spacer1"/>
         <child link="caster_wheel1"/>
-        <origin xyz="0.2 0 -0.02"/>
+        <origin xyz="0 0 -0.0175"/>  <!-- Half spacer length (0.01) + half caster radius (0.0075) -->
     </joint>
     <link name="caster_wheel1">
         <visual>
             <geometry>
-                <sphere radius="0.02"/>
-            </geometry>
-            <material name="black"/>
-        </visual>
-        <collision>
-            <geometry>
-                <sphere radius="0.02"/>
-            </geometry>
-        </collision>
-        <xacro:inertial_sphere mass="0.05" radius="0.02" >
+                <sphere radius="0.0075"/>
+            </geometry>
+            <material name="peacock_dark_blue"/>
+        </visual>
+        <collision>
+            <geometry>
+                <sphere radius="0.0075"/>
+            </geometry>
+        </collision>
+        <xacro:inertial_sphere mass="0.05" radius="0.0075">
             <origin xyz="0 0 0" rpy="0 0 0"/>
         </xacro:inertial_sphere>
     </link>
-    <!--CASTER WHEEL LINK2-->
+    <gazebo reference="caster_wheel1">
+        <material>Gazebo/Purple</material>
+        <mu1 value="0.001"/>
+        <mu2 value="0.001"/>
+    </gazebo>
+    <!--CASTER SPACER 2 - Small cylinder to drop caster down-->
+    <joint name="caster_spacer_joint2" type="fixed">
+        <parent link="chassis"/>
+        <child link="caster_spacer2"/>
+        <origin xyz="0.225 0 -0.0075"/>
+    </joint>
+    <link name="caster_spacer2">
+        <visual>
+            <geometry>
+                <cylinder radius="0.003" length="0.02"/>  <!-- Small spacer: 3mm radius, 20mm length -->
+            </geometry>
+            <material name="grey"/>
+        </visual>
+        <collision>
+            <geometry>
+                <cylinder radius="0.003" length="0.02"/>
+            </geometry>
+        </collision>
+        <xacro:inertial_cylinder mass="0.01" radius="0.003" length="0.02">
+            <origin xyz="0 0 0" rpy="0 0 0"/>
+        </xacro:inertial_cylinder>
+    </link>
+    <gazebo reference="caster_spacer2">
+        <material>Gazebo/Grey</material>
+    </gazebo>
+    <!--CASTER WHEEL LINK2 - Attached to bottom of spacer-->
     <joint name="caster_wheel_joint2" type="fixed">
-        <parent link="chassis"/>
+        <parent link="caster_spacer2"/>
         <child link="caster_wheel2"/>
-        <origin xyz="0.02 0 -0.02"/>
+        <origin xyz="0 0 -0.0175"/>  <!-- Half spacer length (0.01) + half caster radius (0.0075) -->
     </joint>
     <link name="caster_wheel2">
         <visual>
             <geometry>
-                <sphere radius="0.02"/>
-            </geometry>
-            <material name="black"/>
-        </visual>
-        <collision>
-            <geometry>
-                <sphere radius="0.02"/>
-            </geometry>
-        </collision>
-        <xacro:inertial_sphere mass="0.05" radius="0.02" >
+                <sphere radius="0.0075"/>
+            </geometry>
+            <material name="peacock_dark_blue"/>
+        </visual>
+        <collision>
+            <geometry>
+                <sphere radius="0.0075"/>
+            </geometry>
+        </collision>
+        <xacro:inertial_sphere mass="0.05" radius="0.0075">
             <origin xyz="0 0 0" rpy="0 0 0"/>
         </xacro:inertial_sphere>
     </link>
+    <gazebo reference="caster_wheel2">
+        <material>Gazebo/Purple</material>
+        <mu1 value="0.001"/>
+        <mu2 value="0.001"/>
+    </gazebo>
+    <!-- SPACERS - 4 cylindrical supports for upper layer -->
+    <joint name="spacer_joint_1" type="fixed">
+        <parent link="chassis"/>
+        <child link="spacer_1"/>
+        <origin xyz="0.1 0.065 0.02" rpy="0 0 0"/>
+    </joint>
+    <link name="spacer_1">
+        <visual>
+            <geometry>
+                <cylinder radius="0.0007" length="0.04"/>
+            </geometry>
+            <material name="peacock_gold"/>
+        </visual>
+        <collision>
+            <geometry>
+                <cylinder radius="0.0007" length="0.04"/>
+            </geometry>
+        </collision>
+        <xacro:inertial_cylinder mass="0.005" radius="0.0007" length="0.04">
+            <origin xyz="0 0 0" rpy="0 0 0"/>
+        </xacro:inertial_cylinder>
+    </link>
+    <gazebo reference="spacer_1">
+        <material>Gazebo/Turquoise</material>
+    </gazebo>
+    <joint name="spacer_joint_2" type="fixed">
+        <parent link="chassis"/>
+        <child link="spacer_2"/>
+        <origin xyz="0.1 -0.065 0.02" rpy="0 0 0"/>
+    </joint>
+    <link name="spacer_2">
+        <visual>
+            <geometry>
+                <cylinder radius="0.0007" length="0.04"/>
+            </geometry>
+            <material name="peacock_gold"/>
+        </visual>
+        <collision>
+            <geometry>
+                <cylinder radius="0.0007" length="0.04"/>
+            </geometry>
+        </collision>
+        <xacro:inertial_cylinder mass="0.005" radius="0.0007" length="0.04">
+            <origin xyz="0 0 0" rpy="0 0 0"/>
+        </xacro:inertial_cylinder>
+    </link>
+    <gazebo reference="spacer_2">
+        <material>Gazebo/Turquoise</material>
+    </gazebo>
+    <joint name="spacer_joint_3" type="fixed">
+        <parent link="chassis"/>
+        <child link="spacer_3"/>
+        <origin xyz="0.2 0.065 0.02" rpy="0 0 0"/>
+    </joint>
+    <link name="spacer_3">
+        <visual>
+            <geometry>
+                <cylinder radius="0.0007" length="0.04"/>
+            </geometry>
+            <material name="peacock_gold"/>
+        </visual>
+        <collision>
+            <geometry>
+                <cylinder radius="0.0007" length="0.04"/>
+            </geometry>
+        </collision>
+        <xacro:inertial_cylinder mass="0.005" radius="0.0007" length="0.04">
+            <origin xyz="0 0 0" rpy="0 0 0"/>
+        </xacro:inertial_cylinder>
+    </link>
+    <gazebo reference="spacer_3">
+        <material>Gazebo/Turquoise</material>
+    </gazebo>
+    <joint name="spacer_joint_4" type="fixed">
+        <parent link="chassis"/>
+        <child link="spacer_4"/>
+        <origin xyz="0.2 -0.065 0.02" rpy="0 0 0"/>
+    </joint>
+    <link name="spacer_4">
+        <visual>
+            <geometry>
+                <cylinder radius="0.0007" length="0.04"/>
+            </geometry>
+            <material name="peacock_gold"/>
+        </visual>
+        <collision>
+            <geometry>
+                <cylinder radius="0.0007" length="0.04"/>
+            </geometry>
+        </collision>
+        <xacro:inertial_cylinder mass="0.005" radius="0.0007" length="0.04">
+            <origin xyz="0 0 0" rpy="0 0 0"/>
+        </xacro:inertial_cylinder>
+    </link>
+    <gazebo reference="spacer_4">
+        <material>Gazebo/Turquoise</material>
+    </gazebo>
+    <!-- UPPER PLATE -->
+    <joint name="upper_plate_joint" type="fixed">
+        <parent link="chassis"/>
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