Commit message: Updates

File: description/robot_core.xacro (robot description, xacro)
@@ -81,5 +81,5 @@
                 <cylinder radius="0.035" length="0.04"/>
             </geometry>
-            <material name="peacock_dark_blue"/>
+            <material name="black"/>
         </visual>
         <collision>
@@ -93,5 +93,5 @@
     </link>
     <gazebo reference="left_wheel">
-        <material>Gazebo/Purple</material>
+        <material>Gazebo/Black</material>
         <mu1>1.2</mu1>
         <mu2>1.2</mu2>
@@ -111,5 +111,5 @@
                 <cylinder radius="0.035" length="0.04"/>
             </geometry>
-            <material name="peacock_dark_blue"/>
+            <material name="black"/>
         </visual>
         <collision>
@@ -123,5 +123,5 @@
     </link>
     <gazebo reference="right_wheel">
-        <material>Gazebo/Purple</material>
+        <material>Gazebo/Black</material>
         <mu1>1.2</mu1>
         <mu2>1.2</mu2>
@@ -165,5 +165,5 @@
                 <sphere radius="0.0075"/>
             </geometry>
-            <material name="peacock_dark_blue"/>
+            <material name="black"/>
         </visual>
         <collision>
@@ -177,5 +177,5 @@
     </link>
     <gazebo reference="caster_wheel1">
-        <material>Gazebo/Purple</material>
+        <material>Gazebo/Black</material>
         <mu1 value="0.001"/>
         <mu2 value="0.001"/>
@@ -217,5 +217,5 @@
                 <sphere radius="0.0075"/>
             </geometry>
-            <material name="peacock_dark_blue"/>
+            <material name="black"/>
         </visual>
         <collision>
@@ -229,5 +229,5 @@
     </link>
     <gazebo reference="caster_wheel2">
-        <material>Gazebo/Purple</material>
+        <material>Gazebo/Black</material>
         <mu1 value="0.001"/>
         <mu2 value="0.001"/>
